File: RGB-YPbPr-Converter.kicad_sch (KiCad schematic)
At the start: 58 parts, among them J1 Barrel Jack 5.5/2.1, J2 D-Sub HD15 Female, J3 BNC 75 Ohm, J4 BNC 75 Ohm, J5 BNC 75 Ohm, Q1 Q_NPN_BEC, Q2 Q_NPN_BEC, Q3 Q_NPN_BEC, U1 1117-5.0, U2 ICL7660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

Commit message: WIP of sandwich version
Parts:
- removed C1, C6, C7: 10u/16V, Capacitor_THT:CP_Radial_D5.0mm_P2.00mm, symbol Device:C_Polarized_Small
- removed C2, C3, C4, C5, C8, C9: 100n/16V, Capacitor_SMD:C_0805_2012Metric, symbol Device:C_Small
- removed D1: 1N4001, Diode_THT:D_DO-41_SOD81_P10.16mm_Horizontal, symbol Diode:1N4001
- removed D2: 5.6V, Diode_SMD:D_SOD-323_HandSoldering, symbol Device:D_Zener
- removed D3: Green, LED_SMD:LED_0805_2012Metric, symbol Device:LED
- removed J1: Barrel Jack 5.5/2.1, Connector_BarrelJack:BarrelJack_Horizontal, symbol Connector:Barrel_Jack_Switch
- removed J2: D-Sub HD15 Female, lib:ICD15S13E4GV00LF, symbol Connector:DB15_Female_HighDensity_MountingHoles
- removed J3, J4, J5: BNC 75 Ohm, Connector_Coaxial:BNC_Amphenol_B6252HB-NPP3G-50_Horizontal, symbol Connector:Conn_Coaxial
- removed Q1, Q2, Q3: Q_NPN_BEC, Package_TO_SOT_SMD:SOT-23, symbol Device:Q_NPN_BEC
- removed R1, R2, R22, R3, R6, R7: 75, Resistor_SMD:R_0805_2012Metric, symbol Device:R_Small
- removed R10: 549, Resistor_SMD:R_0805_2012Metric, symbol Device:R_Small
- removed R11: 2940, Resistor_SMD:R_0805_2012Metric, symbol Device:R_Small
- removed R12, R13, R14, R18, R25, R26, R28, R30: 0R, Resistor_SMD:R_0805_2012Metric, symbol Device:R_Small
- removed R15, R16, R17, R19, R24, R4, R5, R8: 1k, Resistor_SMD:R_0805_2012Metric, symbol Device:R_Small
- removed R20: 570, Resistor_SMD:R_0805_2012Metric, symbol Device:R_Small
- removed R21: 133, Resistor_SMD:R_0805_2012Metric, symbol Device:R_Small
- removed R23: 105, Resistor_SMD:R_0805_2012Metric, symbol Device:R_Small
- removed R27: 174, Resistor_SMD:R_0805_2012Metric, symbol Device:R_Small
- removed R29: 261, Resistor_SMD:R_0805_2012Metric, symbol Device:R_Small
- removed R9: 1070, Resistor_SMD:R_0805_2012Metric, symbol Device:R_Small
- removed U1: 1117-5.0, Package_TO_SOT_SMD:SOT-223, symbol Regulator_Linear:LM1117-5.0
- removed U2: ICL7660, Package_SO:SOIC-8_3.9x4.9mm_P1.27mm, symbol Regulator_SwitchedCapacitor:ICL7660
- removed U3: LMV793MFX, Package_TO_SOT_SMD:SOT-23-5, symbol Comparator:LMV7219M5
- removed U4: LT6550, Package_SO:MSOP-10_3x3mm_P0.5mm, symbol lib:LT6550
Connections:
- no-connect marks 7 -> 0
Other:
- added sheet Conversion Board (Conversion Board.kicad_sch)
- added sheet Input Board (Input Board.kicad_sch)
- added sheet Output Board (Output Board.kicad_sch)
- note removed: "Based on LT6550 reference design"
- note removed: "Y = 0.229R + 0.587G + 0.114B P_{B} = 0.565(B - Y) P_{R} = 0.713(R - Y)"
- moved on the sheet: H1, H2, H3, H4
