File: RGB-YPbPr-Converter.kicad_sch (KiCad schematic)
At the start: 26 parts, among them J1 RGB, J2 Component, J3 PWR, U1 LMV793MFX, U2 LT6550, U3 ICL7660

Commit message: Add H and V sync pulses to Y channel
Parts:
- added D2: (no value), symbol Device:D_Zener
- added Q1: Q_NPN_BEC, symbol Device:Q_NPN_BEC
- added Q2, Q3: (no value), symbol Device:Q_NPN_BEC
- added R15, R16, R19, R20: (no value), symbol Device:R_Small
- added R17, R18: 1k, symbol Device:R_Small
Connections:
- net +5V: now also R16.1
- net -5V: now also Q1.2 (E), R18.2
- net GND: now also Q3.2 (E)
- net Y: now also R15.2
- net H_SYNC: now reaches J1.13
- net H_SYNC: now also R19.1
- net V_SYNC: now reaches J1.14
- net V_SYNC: now also R20.1
- new net: Q1.1 (B), R17.2, R18.1
- new net: Q1.3 (C), R15.1
- new net: Q3.1 (B), R20.2
- new net: Q2.2 (E), Q3.3 (C)
- new net: Q2.1 (B), R19.2
- new net: D2.1 (K), Q2.3 (C), R16.2
- new net: D2.2 (A), R17.1
- no-connect marks 14 -> 12

Commit message: finished board
Parts:
- removed J2: Component, Connector_Dsub:DSUB-15-HD_Male_Horizontal_P2.29x1.98mm_EdgePinOffset3.03mm_Housed_MountingHolesOffset4.94mm, symbol Connector:DB15_Male_HighDensity_MountingHoles
- removed J3: PWR, TerminalBlock:TerminalBlock_bornier-2_P5.08mm, symbol Connector:Screw_Terminal_01x02
- added C1: 10u/16V, Capacitor_THT:CP_Radial_D5.0mm_P2.00mm, symbol Device:C_Polarized_Small
- added C2, C3, C9: 100n, Capacitor_SMD:C_0805_2012Metric, symbol Device:C_Small
- added D1: 1N4001, Diode_THT:D_DO-41_SOD81_P10.16mm_Horizontal, symbol Diode:1N4001
- added H1, H2, H3, H4: DNP, MountingHole:MountingHole_3.2mm_M3_ISO7380_Pad, symbol Mechanical:MountingHole_Pad
- added J1: Barrel Jack 5.5/2.1, Connector_BarrelJack:BarrelJack_Horizontal, symbol Connector:Barrel_Jack_Switch
- added J3, J4, J5: BNC 75 Ohm, Connector_Coaxial:BNC_Amphenol_B6252HB-NPP3G-50_Horizontal, symbol Connector:Conn_Coaxial
- added R1, R2: 75, Resistor_SMD:R_0805_2012Metric, symbol Device:R_Small
- added R15: 0R, Resistor_SMD:R_0805_2012Metric, symbol Device:R_Small
- added U1: 1117-5.0, Package_TO_SOT_SMD:SOT-223, symbol Regulator_Linear:LM1117-5.0
- C6: renamed from C5; value 10u -> 10u/16V
- C7: renamed from C3; value 10u -> 10u/16V
- D2: value (none) -> 5.6V; footprint (none) -> Diode_SMD:D_SOD-323_HandSoldering; Manufacturer (none) -> Vishay; Part Number (none) -> BZX384-C5V6,115; TME (none) -> BZX384-C5V6.115
- J2: renamed from J1; value RGB -> D-Sub HD15 Female; footprint Connector_Dsub:DSUB-15-HD_Male_Horizontal_P2.29x1.98mm_EdgePinOffset3.03mm_Housed_MountingHolesOffset4.94mm -> lib:ICD15S13E4GV00LF; symbol Connector:DB15_Male_HighDensity_MountingHoles -> Connector:DB15_Female_HighDensity_MountingHoles; Manufacturer (none) -> Amphenol; Part Number (none) -> ICD15S13E4GV00LF; TME (none) -> ICD15S13E4GV00LF
- Q1: renamed from Q2; value (none) -> Q_NPN_BEC; footprint (none) -> Package_TO_SOT_SMD:SOT-23
- Q2: renamed from Q3; value (none) -> Q_NPN_BEC; footprint (none) -> Package_TO_SOT_SMD:SOT-23
- Q3: renamed from Q1; footprint (none) -> Package_TO_SOT_SMD:SOT-23
- R12: renamed from R17; footprint (none) -> Resistor_SMD:R_0805_2012Metric
- R14: renamed from R18; footprint (none) -> Resistor_SMD:R_0805_2012Metric
- R17: renamed from R15; value (none) -> 570; footprint (none) -> Resistor_SMD:R_0805_2012Metric
- R3: renamed from R20; value (none) -> 1k; footprint (none) -> Resistor_SMD:R_0805_2012Metric
- R4: renamed from R19; value (none) -> 1k; footprint (none) -> Resistor_SMD:R_0805_2012Metric
- R8: renamed from R16; value (none) -> 1k; footprint (none) -> Resistor_SMD:R_0805_2012Metric
- U2: renamed from U3; footprint Package_SO:MSOP-8_3x3mm_P0.65mm -> Package_SO:SOIC-8_3.9x4.9mm_P1.27mm; Manufacturer (none) -> Renesas/Intersil; Mouser (none) -> 968-ICL7660AIBAZA; Part Number (none) -> ICL7660AIBAZA; TME (none) -> ICL7660AIBAZA
- U3: renamed from U1; Manufacturer (none) -> Texas Instruments; Mouser (none) -> 926-LMV793MFX/NOPB; Part Number (none) -> LMV793MFX/NOPB
- U4: renamed from U2; Manufacturer (none) -> Analog Devices; Mouser (none) -> LT6550CMS#PBF; Part Number (none) -> LT6550CMS#PBF
- renumbered C1 to C5, C2 to C8, D1 to D3, R5 to R10, R10 to R11, R14 to R13, R13 to R16, R1 to R18, R2 to R19, R11 to R20, R12 to R21, R6 to R22, R3 to R23, R7 to R5, R8 to R6, R9 to R7, R4 to R9
Connections:
- net +5V: now also R18.2, C3.1, R15.2, U1.2 (VO); no longer C5.1, R18.1, U3.5 (V+)
- net -5V: now also C9.2
- net B: now also U4.1 (IN1); no longer U4.3 (IN3)
- net GND: now also D3.1 (K), C1.2, C2.2, C3.2, C9.1, H1.1, H2.1, H3.1, H4.1, J1.2, J1.3, J3.2 (Ext), J4.2 (Ext), J5.2 (Ext), R1.2, R2.2, U1.1 (GND); no longer D3.2 (A), J2.9
- net H_SYNC: now also R2.1
- net Pb: now also R19.2, J3.1 (In); no longer R20.2
- net Pr: now also R20.2, J5.1 (In); no longer R19.2
- net R: now also U4.3 (IN3); no longer U4.1 (IN1)
- net V_SYNC: now also R1.1
- net Y: now also J4.1 (In)
- net Pb_OUT: now reaches R19.1, U4.9 (OUT1)
- net YSUM: now reaches R10.2, R11.2, R9.2, U3.3 (+)
- net FB: now reaches R13.2, R16.1, U3.4 (-)
- net YAMP: now reaches R16.2, U3.1, U4.2 (IN2)
- net H_R: now reaches Q2.1 (B)
- net H_R: now also R4.2; no longer R3.2
- net CAP+: now reaches C6.1, U2.2 (CAP+)
- net CAP-: now reaches C6.2, U2.4 (CAP-)
- net Pr_OUT: now reaches R20.1, U4.7 (OUT3)
- net V_R: now reaches Q1.1 (B)
- net V_R: now also R3.2; no longer R4.2
- net Y_FB renamed Y_OUT
- new net: D3.2 (A), R18.1
- new net +5VAMP: C5.1, R15.1, U3.5 (V+)
- new net VIN: D1.2 (A), J1.1
- new net VIND: C1.1, C2.1, D1.1 (K), U1.3 (VI)
- no-connect marks 12 -> 7
Other:
- moved on the sheet: C4, C5, C6, C7, C8, D3, R13, R16, R18, R19, R20, R21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

Commit message: fixes
Parts:
- added R12, R13, R14, R25, R26, R28, R30: 0R, Resistor_SMD:R_0805_2012Metric, symbol Device:R_Small
- C1, C6, C7: Manufacturer (none) -> Generic; Part Number (none) -> 10u/16V; TME (none) -> UVR1C100MDD
- C2, C3, C4, C5, C8, C9: value 100n -> 100n/16V; Manufacturer (none) -> Generic; Part Number (none) -> 100n/16V
- D3: value PWR -> Green; Manufacturer (none) -> Generic; Part Number (none) -> LED 0805 Green; TME (none) -> LTST-C170KGKT
- Q1, Q2, Q3: Manufacturer (none) -> Generic; Part Number (none) -> BC847C; TME (none) -> BC847C.215
- R21: renamed from R19; value 105 -> 133
- R22: value 105 -> 75
- renumbered R12 to R15, R13 to R16, R14 to R17, R15 to R18, R16 to R19, R17 to R20, R20 to R23, R18 to R24, R21 to R27, R23 to R29, R5 to R3, R3 to R4, R4 to R5
Connections:
- net GND: now also R28.2, R30.2; no longer R27.2, R29.2
- net Pb: now also R25.2; no longer R21.2
- net Pr: now also R26.2; no longer R23.2
- net YSUM: now also R12.2, R13.2, R14.2; no longer R10.2, R11.2, R9.2
- new net: R12.1, R9.2
- new net: R27.2, R28.1
- new net: R21.2, R25.1
- new net: R11.2, R14.1
- new net: R10.2, R13.1
- new net: R29.2, R30.1
- new net: R23.2, R26.1
Other:
- moved on the sheet: R10, R11, R21, R22, R23, R27, R29, R3, R6, R7, R9

Commit message: emergency version for decrunch 2023
Parts:
- removed C6, C7: 10u/16V, Capacitor_THT:CP_Radial_D5.0mm_P2.00mm, symbol Device:C_Polarized_Small
- removed D1: 1N4001, Diode_THT:D_DO-41_SOD81_P10.16mm_Horizontal, symbol Diode:1N4001
- removed R1, R2: 75, Resistor_SMD:R_0805_2012Metric, symbol Device:R_Small
- removed R18: 0R, Resistor_SMD:R_0805_2012Metric, symbol Device:R_Small
- removed U2: ICL7660, Package_SO:SOIC-8_3.9x4.9mm_P1.27mm, symbol Regulator_SwitchedCapacitor:ICL7660
- removed U3: LMV793MFX, Package_TO_SOT_SMD:SOT-23-5, symbol Comparator:LMV7219M5
- added C6: 100n/16V, Capacitor_SMD:C_0805_2012Metric, symbol Device:C_Small
- added U2: 1117-5.0, Package_TO_SOT_SMD:SOT-223, symbol Regulator_Linear:LM1117-5.0
- added U5: AD818ARZ, Package_SO:SO-8_3.9x4.9mm_P1.27mm, symbol lib:AD818ARZ
- R24: value 1k -> 10k
Connections:
- net +5VAMP is gone; now on net +5V: C5.1
- net VIND is gone; now on net VIN: C1.1, C2.1, U1.3 (VI)
- net +5V: now also U2.2 (VO), U5.7 (+VS); no longer C3.1, R24.2, U1.2 (VO)
- net -5V: now also C1.2, C2.2, C3.2, C5.2, D3.1 (K), J1.2, J1.3, U1.1 (GND), U5.4 (-VS)
- net FB: now also U5.2 (-IN)
- net GND: now also C3.1, U1.2 (VO), C6.2, U2.1 (GND); no longer C1.2, C2.2, C3.2, C5.2, D3.1 (K), J1.2, J1.3, U1.1 (GND)
- net VIN: now also R24.2, C6.1, U2.3 (VI)
- net YAMP: now also U5.6 (OUT)
- net YSUM: now also U5.3 (+IN)
Other:
- moved on the sheet: C1, C2, C3, C5, D3, J1, J2, R10, R11, R12, R13, R14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

Commit message: gerbers + resistor values
Parts:
- R10: value 549 -> 510
- R11: value 2940 -> 2700
- R12: value 0R -> 510
- R13, R30: value 0R -> 39
- R14: value 0R -> 220
- R20: value 570 -> 560
- R21: value 133 -> 120
- R23: value 105 -> 100
- R25: value 0R -> 12
- R26: value 0R -> 3.9
- R27: value 174 -> 120
- R28: value 0R -> 51
- R29: value 261 -> 220
- R9: value 1070 -> 560
- U4: Mouser LT6550CMS#PBF -> (none)
- U5: Manufacturer (none) -> Analog Devices; OC_FARNELL 2131892 -> (none); Part Number (none) -> AD818ARZ
Other:
- note added: "105"
- note added: "1070"
- note added: "133"
- note added: "174"
- note added: "261"
- note added: "2940"
- note added: "549"
- note added: "570"
Changed lines of the file:
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@@
+    (effects (font (size 1.27 1.27)) (justify left bottom))
+  )
+  (text "1070" (at 76.962 88.138 0)
+    (effects (font (size 1.27 1.27)) (justify left bottom))
+  )
+  (text "174" (at 219.202 88.138 0)
+    (effects (font (size 1.27 1.27)) (justify left bottom))
+  )
+  (text "105" (at 191.262 120.904 0)
+    (effects (font (size 1.27 1.27)) (justify left bottom))
+  )
+  (text "570" (at 131.572 143.51 0)
+    (effects (font (size 1.27 1.27)) (justify left bottom))
+  )
+  (text "261" (at 218.948 125.984 0)
+    (effects (font (size 1.27 1.27)) (justify left bottom))
+  )
+  (text "2940" (at 77.47 103.886 0)
+    (effects (font (size 1.27 1.27)) (justify left bottom))
+  )
+  (text "133" (at 190.5 79.756 0)
     (effects (font (size 1.27 1.27)) (justify left bottom))
   )
@@
     (effects (font (size 1.27 1.27)) (justify left bottom))
   )
+  (text "549" (at 76.962 95.758 0)
+    (effects (font (size 1.27 1.27)) (justify left bottom))
+  )
   (label "R" (at 153.67 101.6 0) (fields_autoplaced)
     (effects (font (size 1.27 1.27)) (justify left bottom))
@@
       (effects (font (size 1.27 1.27)))
     )
-    (property "Value" "0R" (at 92.71 86.36 90)
+    (property "Value" "510" (at 92.71 86.36 90)
       (effects (font (size 1.27 1.27)))
     )
@@
   (symbol (lib_id "Device:R_Small") (at 139.7 144.78 90) (unit 1)
     (in_bom yes) (on_board yes) (dnp no) (fields_autoplaced)
-    (property "Reference" "R20" (at 139.7 138.43 90)
-      (effects (font (size 1.27 1.27)))
-    )
-    (property "Value" "570" (at 139.7 140.97 90)
+    (property "Reference" "R20" (at 139.7 139.7 90)
+      (effects (font (size 1.27 1.27)))
+    )
+    (property "Value" "560" (at 139.7 142.24 90)
       (effects (font (size 1.27 1.27)))
     )
@@
   (symbol (lib_id "Device:R_Small") (at 211.455 90.17 0) (unit 1)
     (in_bom yes) (on_board yes) (dnp no) (fields_autoplaced)
-    (property "Reference" "R28" (at 213.36 88.8999 0)
-      (effects (font (size 1.27 1.27)) (justify left))
-    )
-    (property "Value" "0R" (at 213.36 91.4399 0)
+    (property "Reference" "R28" (at 213.36 89.535 0)
+      (effects (font (size 1.27 1.27)) (justify left))
+    )
+    (property "Value" "51" (at 213.36 92.075 0)
       (effects (font (size 1.27 1.27)) (justify left))
     )
@@
       (effects (font (size 1.27 1.27)))
     )
-    (property "Value" "133" (at 198.12 77.47 90)
+    (property "Value" "120" (at 198.12 77.47 90)
       (effects (font (size 1.27 1.27)))
     )
@@
       (effects (font (size 1.27 1.27)))
     )
-    (property "Value" "0R" (at 92.71 101.6 90)
+    (property "Value" "220" (at 92.71 101.6 90)
       (effects (font (size 1.27 1.27)))
     )
@@
       (effects (font (size 1.27 1.27)))
     )
-    (property "Value" "0R" (at 205.105 77.47 90)
+    (property "Value" "12" (at 205.105 77.47 90)
       (effects (font (size 1.27 1.27)))
     )
@@
       (effects (font (size 1.27 1.27)))
     )
-    (property "Value" "2940" (at 84.455 101.6 90)
+    (property "Value" "2700" (at 84.455 101.6 90)
       (effects (font (size 1.27 1.27)))
     )
@@
       (effects (font (size 1.27 1.27)))
     )
-    (property "Value" "1070" (at 84.455 86.36 90)
+    (property "Value" "560" (at 84.455 86.36 90)
       (effects (font (size 1.27 1.27)))
     )
@@
     )
     (property "Manufacturer" "Analog Devices" (at 167.64 99.06 0)
-      (effects (font (size 1.27 1.27)) hide)
-    )
-    (property "Mouser" "LT6550CMS#PBF" (at 167.64 99.06 0)
       (effects (font (size 1.27 1.27)) hide)
     )
@@
       (effects (font (size 1.27 1.27)) hide)
     )
-    (property "OC_FARNELL" "2131892" (at 214.4056 87.287 0)
-      (effects (font (size 1.27 1.27)) (justify bottom) hide)
+    (property "Manufacturer" "Analog Devices" (at 187.706 45.974 0)
+      (effects (font (size 1.27 1.27)) hide)
+    )
+    (property "Part Number" "AD818ARZ" (at 187.706 45.974 0)
+      (effects (font (size 1.27 1.27)) hide)
     )
     (pin "1")
@@
       (effects (font (size 1.27 1.27)))
     )
-    (property "Value" "549" (at 84.455 93.98 90)
+    (property "Value" "510" (at 84.455 93.98 90)
       (effects (font (size 1.27 1.27)))
     )
@@
       (effects (font (size 1.27 1.27)) (justify left))
     )
-    (property "Value" "174" (at 213.995 85.0899 0)
+    (property "Value" "120" (at 213.995 85.0899 0)
       (effects (font (size 1.27 1.27)) (justify left))
     )
@@
       (effects (font (size 1.27 1.27)))
     )
-    (property "Value" "0R" (at 92.71 93.98 90)
+    (property "Value" "39" (at 92.71 93.98 90)
       (effects (font (size 1.27 1.27)))
     )
@@
   (symbol (lib_id "Device:R_Small") (at 211.455 128.27 0) (unit 1)
     (in_bom yes) (on_board yes) (dnp no) (fields_autoplaced)
-    (property "Reference" "R30" (at 213.36 126.9999 0)
-      (effects (font (size 1.27 1.27)) (justify left))
-    )
-    (property "Value" "0R" (at 213.36 129.5399 0)
+    (property "Reference" "R30" (at 213.36 127.635 0)
+      (effects (font (size 1.27 1.27)) (justify left))
+    )
+    (property "Value" "39" (at 213.36 130.175 0)
       (effects (font (size 1.27 1.27)) (justify left))
     )
@@
       (effects (font (size 1.27 1.27)))
     )
-    (property "Value" "105" (at 198.12 115.57 90)
+    (property "Value" "100" (at 198.12 115.57 90)
       (effects (font (size 1.27 1.27)))
     )
@@
       (effects (font (size 1.27 1.27)))
     )
-    (property "Value" "0R" (at 205.105 115.57 90)
+    (property "Value" "3.9" (at 205.105 115.57 90)
       (effects (font (size 1.27 1.27)))
     )
@@
       (effects (font (size 1.27 1.27)) (justify left))
     )
-    (property "Value" "261" (at 213.995 123.1899 0)
-      (effects (font (size 1.27 1.27)) (justify left))
-    )
+    (property "Value" "220" (at 213.995 123.1899 0)
+      (effects (font (size 1.27 1.27)) (justify left))
+    )
