File: RGB-YPbPr-Converter.kicad_sch (KiCad schematic)
At the start: 4 parts

Commit message: WIP
Parts:
- removed H1, H2, H3, H4: DNP, MountingHole:MountingHole_3.2mm_M3_ISO7380_Pad, symbol Mechanical:MountingHole_Pad
- added J6: Conn_01x05_Male, Connector_PinHeader_2.54mm:PinHeader_1x05_P2.54mm_Vertical, symbol Connector:Conn_01x05_Male
- added J7: Conn_01x05_Female, Connector_PinSocket_2.54mm:PinSocket_1x05_P2.54mm_Vertical, symbol Connector:Conn_01x05_Female
- added J8: Conn_01x03_Male, Connector_PinHeader_2.54mm:PinHeader_1x03_P2.54mm_Vertical, symbol Connector:Conn_01x03_Male
- added J9: Conn_01x03_Female, Connector_PinSocket_2.54mm:PinSocket_1x03_P2.54mm_Vertical, symbol Connector:Conn_01x03_Female
Connections:
- net Conversion Board/B: now also J6.4 (Pin_4), J7.4 (Pin_4)
- net Conversion Board/G: now also J6.2 (Pin_2), J7.2 (Pin_2)
- net Conversion Board/R: now also J6.1 (Pin_1), J7.1 (Pin_1)
- net Conversion Board/SYNC: now also J6.5 (Pin_5), J7.5 (Pin_5)
- net GND: now also J6.3 (Pin_3), J7.3 (Pin_3)
- new net Input Board/+5V: J8.1 (Pin_1), J9.1 (Pin_1)
- new net Input Board/-5V: J8.3 (Pin_3), J9.3 (Pin_3)
- new net Input Board/GND: J8.2 (Pin_2), J9.2 (Pin_2)
Other:
- sheet Input Board ports: added +5V, -5V, GND; removed none

Commit message: WIP
Parts:
- removed J6: Conn_01x05_Male, Connector_PinHeader_2.54mm:PinHeader_1x05_P2.54mm_Vertical, symbol Connector:Conn_01x05_Male
- removed J7: Conn_01x05_Female, Connector_PinSocket_2.54mm:PinSocket_1x05_P2.54mm_Vertical, symbol Connector:Conn_01x05_Female
- removed J8: Conn_01x03_Male, Connector_PinHeader_2.54mm:PinHeader_1x03_P2.54mm_Vertical, symbol Connector:Conn_01x03_Male
- removed J9: Conn_01x03_Female, Connector_PinSocket_2.54mm:PinSocket_1x03_P2.54mm_Vertical, symbol Connector:Conn_01x03_Female
- added J10, J12, J6, J8: 690357101072, lib:690357101072, symbol 690357101072:690357101072
- added J11, J13, J7, J9: 690367181072, lib:690367181072, symbol 690367181072:690367181072
