File: Input Board.kicad_sch (KiCad schematic)
At the start: 24 parts, among them J1 ADC-010-1, J2 D-Sub HD15 Female, Q1 BC847C, Q2 BC847C, Q3 BC847C, U1 L7805, U2 ICL7660, U5 L7905

Commit message: add more 3D models
Parts:
- removed D1: Diode SMA, Diode_SMD:D_SMA, symbol Diode:1N4001
Connections:
- net VIN is gone; now on net +12V: J1.1
Changed lines of the file:
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@@
-    (stroke (width 0) (type default) (color 0 0 0 0))
-  )
-  (wire (pts (xy 93.98 41.91) (xy 83.82 41.91))
     (stroke (width 0) (type default) (color 0 0 0 0))
   )
@@
     (stroke (width 0) (type default) (color 0 0 0 0))
   )
-  (wire (pts (xy 72.39 41.91) (xy 76.2 41.91))
+  (wire (pts (xy 72.39 41.91) (xy 93.98 41.91))
     (stroke (width 0) (type default) (color 0 0 0 0))
   )
@@
   (label "CAP-" (at 140.97 88.9 180)
     (effects (font (size 1.27 1.27)) (justify right bottom))
-  )
-  (label "VIN" (at 73.66 41.91 0)
-    (effects (font (size 1.27 1.27)) (justify left bottom))
   )
   (label "G" (at 90.17 132.08 180)
@@
       (effects (font (size 1.27 1.27)) hide)
     )
-    (pin "1")
-    (pin "2")
-  )
-  (symbol (lib_id "Diode:1N4001") (at 80.01 41.91 180) (unit 1)
-    (in_bom yes) (on_board yes) (fields_autoplaced)
-    (property "Reference" "D1" (id 0) (at 80.01 35.56 0))
-    (property "Value" "Diode SMA" (id 1) (at 80.01 38.1 0))
-    (property "Footprint" "Diode_SMD:D_SMA" (id 2) (at 80.01 37.465 0)
-      (effects (font (size 1.27 1.27)) hide)
-    )
-    (property "Datasheet" "" (id 3) (at 80.01 41.91 0)
-      (effects (font (size 1.27 1.27)) hide)
-    )
-    (property "Manufacturer" "" (id 4) (at 80.01 41.91 0)
-      (effects (font (size 1.27 1.27)) hide)
-    )
-    (property "Part Number" "" (id 5) (at 80.01 41.91 0)
-      (effects (font (size 1.27 1.27)) hide)
-    )
-    (property "TME" "" (id 6) (at 80.01 41.91 0)
-      (effects (font (size 1.27 1.27)) hide)
-    )

Commit message: WIP
Changed lines of the file:
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@@
+    (stroke (width 0) (type default) (color 0 0 0 0))
+  )
+  (wire (pts (xy 195.58 77.47) (xy 195.58 73.66))
     (stroke (width 0) (type default) (color 0 0 0 0))
   )
@@
     (stroke (width 0) (type default) (color 0 0 0 0))
   )
+  (wire (pts (xy 195.58 38.1) (xy 195.58 41.91))
+    (stroke (width 0) (type default) (color 0 0 0 0))
+  )
   (wire (pts (xy 85.09 129.54) (xy 85.09 134.62))
     (stroke (width 0) (type default) (color 0 0 0 0))
@@
     (stroke (width 0) (type default) (color 0 0 0 0))
   )
+  (wire (pts (xy 199.39 58.42) (xy 195.58 58.42))
+    (stroke (width 0) (type default) (color 0 0 0 0))
+  )
   (wire (pts (xy 72.39 44.45) (xy 73.66 44.45))
     (stroke (width 0) (type default) (color 0 0 0 0))
@@
     (stroke (width 0) (type default) (color 0 0 0 0))
   )
+  (wire (pts (xy 199.39 77.47) (xy 195.58 77.47))
+    (stroke (width 0) (type default) (color 0 0 0 0))
+  )
   (wire (pts (xy 173.99 71.12) (xy 173.99 73.66))
+    (stroke (width 0) (type default) (color 0 0 0 0))
+  )
+  (wire (pts (xy 199.39 38.1) (xy 195.58 38.1))
     (stroke (width 0) (type default) (color 0 0 0 0))
   )
@@
     (effects (font (size 1.27 1.27)) (justify left bottom))
   )
+  (hierarchical_label "+5V" (shape output) (at 199.39 38.1 0)
+    (effects (font (size 1.27 1.27)) (justify left))
+  )
   (hierarchical_label "G" (shape output) (at 90.17 132.08 0)
     (effects (font (size 1.27 1.27)) (justify left))
   )
   (hierarchical_label "R" (shape output) (at 90.17 137.16 0)
+    (effects (font (size 1.27 1.27)) (justify left))
+  )
+  (hierarchical_label "-5V" (shape output) (at 199.39 77.47 0)
+    (effects (font (size 1.27 1.27)) (justify left))
+  )
+  (hierarchical_label "GND" (shape output) (at 199.39 58.42 0)
     (effects (font (size 1.27 1.27)) (justify left))
   )
@@
       (effects (font (size 1.27 1.27)) hide)
     )
+    (pin "1")
+  )
+  (symbol (lib_id "power:GND") (at 195.58 58.42 270) (unit 1)
+    (in_bom yes) (on_board yes) (fields_autoplaced)
+    (property "Reference" "#PWR0111" (id 0) (at 189.23 58.42 0)
+      (effects (font (size 1.27 1.27)) hide)
+    )
+    (property "Value" "GND" (id 1) (at 191.77 58.4199 90)
+      (effects (font (size 1.27 1.27)) (justify right))
+    )
+    (property "Footprint" "" (id 2) (at 195.58 58.42 0)
+      (effects (font (size 1.27 1.27)) hide)
+    )
+    (property "Datasheet" "" (id 3) (at 195.58 58.42 0)
+      (effects (font (size 1.27 1.27)) hide)
+    )

Commit message: WIP
Parts:
- added J14: L77HDEH15SOL2RM8C309, lib:AMPHENOL_L77HDEH15SOL2RM8C309, symbol L77HDEH15SOL2RM8C309:L77HDEH15SOL2RM8C309
Connections:
- new net: J14.S1 (SHIELD), J14.S2 (SHIELD)
Other:
- note added: "https://www.tme.eu/pl/details/adc-010-1/zlacza-dc/adam-tech/ 694106402002"
- note removed: "TODO: https://www.tme.eu/pl/details/adc-010-1/zlacza-dc/adam-tech/"
Changed lines of the file:
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@@
     (stroke (width 0) (type default) (color 0 0 0 0))
   )
-  (text "TODO:\nhttps://www.tme.eu/pl/details/adc-010-1/zlacza-dc/adam-tech/"
+  (text "https://www.tme.eu/pl/details/adc-010-1/zlacza-dc/adam-tech/\n694106402002"
     (at 34.29 31.75 0)
     (effects (font (size 1.27 1.27)) (justify left bottom))
@@
     (pin "2")
   )
+  (symbol (lib_id "L77HDEH15SOL2RM8C309:L77HDEH15SOL2RM8C309") (at 110.49 114.3 0) (unit 1)
+    (in_bom yes) (on_board yes) (fields_autoplaced)
+    (property "Reference" "J14" (id 0) (at 110.49 96.52 0))
+    (property "Value" "L77HDEH15SOL2RM8C309" (id 1) (at 110.49 99.06 0))
+    (property "Footprint" "lib:AMPHENOL_L77HDEH15SOL2RM8C309" (id 2) (at 110.49 114.3 0)
+      (effects (font (size 1.27 1.27)) (justify bottom) hide)
+    )
+    (property "Datasheet" "" (id 3) (at 110.49 114.3 0)
+      (effects (font (size 1.27 1.27)) hide)
+    )
+    (property "MAXIMUM_PACKAGE_HEIGHT" "12.2 mm" (id 4) (at 110.49 114.3 0)
+      (effects (font (size 1.27 1.27)) (justify bottom) hide)
+    )
+    (property "PARTREV" "1" (id 5) (at 110.49 114.3 0)
+      (effects (font (size 1.27 1.27)) (justify bottom) hide)
+    )
+    (property "MANUFACTURER" "Amphenol" (id 6) (at 110.49 114.3 0)
+      (effects (font (size 1.27 1.27)) (justify bottom) hide)
+    )
+    (property "STANDARD" "Manufacturer Recommendations" (id 7) (at 110.49 114.3 0)
+      (effects (font (size 1.27 1.27)) (justify bottom) hide)
+    )
+    (pin "1")
+    (pin "10")
+    (pin "11")
+    (pin "12")
+    (pin "13")
+    (pin "14")
+    (pin "15")
+    (pin "2")
+    (pin "3")
+    (pin "4")
+    (pin "5")
+    (pin "6")
+    (pin "7")
+    (pin "8")
+    (pin "9")
+    (pin "S1")
+    (pin "S2")
+  )
   (symbol (lib_id "power:GND") (at 173.99 66.04 180) (unit 1)
